File: HARDWARE/ESP32-PoE-hardware-revision-C1/ESP32-PoE_Rev_C.sch (KiCad schematic (older format))
At the start: 121 parts, among them Q1 Q12MHz/20pF/10ppm/4P/3.2x2.5mm, Q2 BC817-40(SOT23), Q3 BC817-40(SOT23), T1 DTC114YKA(SOT-23), U1 CH340T(SSOP20W), U3 BL4054B-42TPRN(SOT23-5), U4 LAN8710A-EZC(QFN32), U7 SY8089AAAC(SOT23-5), U8 Si3402-B-GM(QFN-20_5x5mm), U9 ESP-WROOM-32

Commit message: Update
Parts:
- removed C19: 22uF/6.3V/20%/X5R/C0603, OLIMEX_RLC-FP:C_0603_5MIL_DWS, symbol ESP32-PoE-ISO_Rev_A:C
- removed C20, C23: NA(1.0nF/3kV/10%/X7R/SMD/1808(VISHAY-VJ1808Y102KB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, OLIMEX_RLC-FP:C_1808(4520)_5MIL_DWS_ISO, symbol ESP32-PoE-ISO_Rev_A:C
- removed C28: 1nF/50V/10%/X7R/C0402, OLIMEX_RLC-FP:C_0402_5MIL_DWS, symbol ESP32-PoE-ISO_Rev_A:C
- removed DCDC1: F0505S-3WR2(SIP-7), OLIMEX_Regulators-FP:SIP-7_Universal, symbol ESP32-PoE-ISO_Rev_A:F0505S-2WR2_AM1D-0505S-NZ(SIP-7_Universal)
- removed R16, R7: 470k/R0402, OLIMEX_RLC-FP:R_0402_5MIL_DWS, symbol ESP32-PoE-ISO_Rev_A:R
- added EN_CT1, EN_CT2: Closed, OLIMEX_Jumpers-FP:SJ_1_SMALLER_TIED, symbol ESP32-PoE_Rev_C:SJ_Closed
- added R7: 0R(board_mounted), OLIMEX_RLC-FP:0R_0603, symbol ESP32-PoE_Rev_C:R
- ACT1, CHRG1, LNK1, PWR1: symbol ESP32-PoE-ISO_Rev_A:LED -> ESP32-PoE_Rev_C:LED
- BAT1: symbol ESP32-PoE-ISO_Rev_A:BAT_CON -> ESP32-PoE_Rev_C:BAT_CON
- BUT1, RST1: symbol ESP32-PoE-ISO_Rev_A:SIDE_WTCM-TR(3x4) -> ESP32-PoE_Rev_C:SIDE_WTCM-TR(3x4)
- C1, C10, C11, C12, C13, C14, C15, C16, C17, C18, C2, C21, C22, C24, C25, C3, C30, C4, C5, C6, C7, C8, C9: symbol ESP32-PoE-ISO_Rev_A:C -> ESP32-PoE_Rev_C:C
- C26: value 1nF/50V/10%/X7R/C0402 -> 1nF/50V/10%/X7R/C0603; footprint OLIMEX_RLC-FP:C_0402_5MIL_DWS -> OLIMEX_RLC-FP:C_0603_5MIL_DWS; symbol ESP32-PoE-ISO_Rev_A:C -> ESP32-PoE_Rev_C:C
- C27: footprint OLIMEX_RLC-FP:CPOL-RM2.5mm_6.3x11mm_PTH -> OLIMEX_RLC-FP:CPOL-RM2.5mm_6.3x11mm_SMD; symbol ESP32-PoE-ISO_Rev_A:CP -> ESP32-PoE_Rev_C:CP
- C29: footprint OLIMEX_RLC-FP:CPOL-RM3.5mm_8.0x11.5mm_PTH -> OLIMEX_RLC-FP:CPOL-RM3.5mm_8.0x11.5mm_SMD; symbol ESP32-PoE-ISO_Rev_A:CP -> ESP32-PoE_Rev_C:CP
- D1, D3: value 1N5819S4/SOD123 -> 1N5822/SS34/SMA; footprint OLIMEX_Diodes-FP:SOD-123_1C-2A_KA -> OLIMEX_Diodes-FP:SMA-KA; symbol ESP32-PoE-ISO_Rev_A:D_Schottky -> ESP32-PoE_Rev_C:D_Schottky
- D2: symbol ESP32-PoE-ISO_Rev_A:BAT54C(SOT23-3) -> ESP32-PoE_Rev_C:BAT54C(SOT23-3)
- D4: value 1N5819S4/SOD-123 -> 1N5819S4(SOD-123); symbol ESP32-PoE-ISO_Rev_A:D_Schottky_Small -> ESP32-PoE_Rev_C:D_Schottky_Small
- D5: symbol ESP32-PoE-ISO_Rev_A:D_Schottky_Small -> ESP32-PoE_Rev_C:D_Schottky_Small
- EXT1, EXT2: symbol ESP32-PoE-ISO_Rev_A:CON10 -> ESP32-PoE_Rev_C:CON10
- FET1, FET2, FET3: symbol ESP32-PoE-ISO_Rev_A:P-MOS+DIOD -> ESP32-PoE_Rev_C:P-MOS+DIOD
- FID1, FID2, FID3, FID4, FID5, FID6: symbol ESP32-PoE-ISO_Rev_A:Fiducial -> ESP32-PoE_Rev_C:Fiducial
- L1, L3, L4, L5, L6: symbol ESP32-PoE-ISO_Rev_A:L -> ESP32-PoE_Rev_C:L
- L2: value 2.2uH/1.5A/DCR=72mR/20%/3.00x3.00x1.50mm/CD32(NR3015T2R2M) -> 2.2uH/1.5A/DCR<0.1R/CD32; symbol ESP32-PoE-ISO_Rev_A:L -> ESP32-PoE_Rev_C:L
- LAN_CON1: value RJP-003TC1(LPJ4112CNL)---Pin<7>_and_<8>_to_be_CUT!!! -> RJP-003TC1(LPJ4112CNL); footprint OLIMEX_Connectors-FP:RJP-003TC1(LPJ4112CNL)-ISO(Pin(7)and(8)CUT) -> OLIMEX_Connectors-FP:RJP-003TC1(LPJ4112CNL); symbol ESP32-PoE-ISO_Rev_A:RJP-003TC1(LPJ4112CNL) -> ESP32-PoE_Rev_C:RJP-003TC1(LPJ4112CNL)-OLIMEX_Connectors
- MICRO_SD1: symbol ESP32-PoE-ISO_Rev_A:MICRO_SD(TFC-9P-1.xH(ATFFS150A01BR016)) -> ESP32-PoE_Rev_C:MICRO_SD(TFC-9P-1.xH(ATFFS150A01BR016))
- Q1: symbol ESP32-PoE-ISO_Rev_A:Crystal_GND -> ESP32-PoE_Rev_C:Crystal_GND
- Q2, Q3: symbol ESP32-PoE-ISO_Rev_A:Q_NPN_BEC -> ESP32-PoE_Rev_C:Q_NPN_BEC
- R1, R10, R11, R12, R13, R14, R15, R18, R19, R2, R20, R21, R24, R25, R26, R3, R31, R32, R33, R34, R35, R36, R37, R38, R39, R4, R40, R41, R42, R43, R44, R45, R46, R47, R48, R49, R5, R8, R9: symbol ESP32-PoE-ISO_Rev_A:R -> ESP32-PoE_Rev_C:R
- R29: value 220k/R0402 -> 4.99k/1%/R0402; symbol ESP32-PoE-ISO_Rev_A:R -> ESP32-PoE_Rev_C:R
- R30: value 49.9k/1%/R0402 -> 1.1k/1%/R0402; symbol ESP32-PoE-ISO_Rev_A:R -> ESP32-PoE_Rev_C:R
- R6: value 3.3k/R0402 -> 2.2k/R0402; symbol ESP32-PoE-ISO_Rev_A:R -> ESP32-PoE_Rev_C:R
- RM1, RM2, RM3: symbol ESP32-PoE-ISO_Rev_A:RA1206_(4x0603)_4B8_Smashed -> ESP32-PoE_Rev_C:RA1206_(4x0603)_4B8_Smashed
- T1: symbol ESP32-PoE-ISO_Rev_A:DTC114YKA(SOT-23) -> ESP32-PoE_Rev_C:DTC114YKA(SOT-23)
- U1: symbol ESP32-PoE-ISO_Rev_A:CH340T(SSOP20W) -> ESP32-PoE_Rev_C:CH340T(SSOP20W)
- U3: symbol ESP32-PoE-ISO_Rev_A:BL4054B-42TPRN(SOT23-5) -> ESP32-PoE_Rev_C:BL4054B-42TPRN(SOT23-5)
- U4: symbol ESP32-PoE-ISO_Rev_A:LAN8710A-EZC(QFN32) -> ESP32-PoE_Rev_C:LAN8710A-EZC(QFN32)
- U7: symbol ESP32-PoE-ISO_Rev_A:SY8009AAAC(SOT23-5) -> ESP32-PoE_Rev_C:SY8009AAAC(SOT23-5)
- U8: symbol ESP32-PoE-ISO_Rev_A:Si3402-B-GM(QFN-20_5x5mm) -> ESP32-PoE_Rev_C:Si3402-B-GM(QFN-20_5x5mm)
- U9: symbol ESP32-PoE-ISO_Rev_A:ESP-WROOM-32 -> ESP32-PoE_Rev_C:ESP-WROOM-32
- UEXT1: value P-B-V-10-LF -> B-V-10-LF(GBH254SMT-10); symbol ESP32-PoE-ISO_Rev_A:BH10S -> ESP32-PoE_Rev_C:BH10S
- USB-UART1: symbol ESP32-PoE-ISO_Rev_A:USB-MINI -> ESP32-PoE_Rev_C:USB-MINI
Connections:
- net labels removed: RD+, RD-, Shield, TD+, TD-, USB_D+, USB_D-, Vneg, Vpos, Vss
- wire segments 559 -> 532
- no-connect marks 22 -> 20
Other:
- note added: "!!!WARNING!!!\nWhen the board is powered via PoE, don't include the USB cable for to programming it!!!\nIn case this is required, USB-ISO must be used for to guarantee galvanic isolation!\nSee: https://www.olimex.com/Products/USB-Modules/USB-ISO/"
- note added: "IBAT = 1000/Rprog = 455mA"
- note added: "Vneg"
- note added: "Vpos"
- note added: "Vss"
- note removed: "Battery\nMeasurement"
- note removed: "Galvanic Isolated Part"
- note removed: "IBAT = 1000/Rprog = 303mA"
- note removed: "Pin 7 and 8 are cut for to \nensure galvanic isolation!!!"
